File: pcb/RadaxZeroLcd.kicad_sch (KiCad schematic)
At the start: 7 parts, among them J1 RadaxZero, J2 4.0inch LCD, J3 UART, J4 I2C, J5 SYS UART

Commit message: update radxa zero footprint
Parts:
- J1: footprint Connector_PinHeader_2.54mm:PinHeader_2x20_P2.54mm_Vertical -> Connector_PinSocket_2.54mm:PinSocket_2x20_P2.54mm_Vertical
Changed lines of the file:
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@@
     (property "Reference" "J1" (id 0) (at 152.4 33.02 0))
     (property "Value" "RadaxZero" (id 1) (at 152.4 35.56 0))
-    (property "Footprint" "Connector_PinHeader_2.54mm:PinHeader_2x20_P2.54mm_Vertical" (id 2) (at 151.13 39.37 0)
+    (property "Footprint" "Connector_PinSocket_2.54mm:PinSocket_2x20_P2.54mm_Vertical" (id 2) (at 151.13 39.37 0)
       (effects (font (size 1.27 1.27)) hide)
     )
@@
     )
     (path "/c31d3e5c-66d2-42fe-ac5a-592c71a1ddb9"
-      (reference "J1") (unit 1) (value "RadaxZero") (footprint "Connector_PinHeader_2.54mm:PinHeader_2x20_P2.54mm_Vertical")
+      (reference "J1") (unit 1) (value "RadaxZero") (footprint "Connector_PinSocket_2.54mm:PinSocket_2x20_P2.54mm_Vertical")
     )
     (path "/9dc01ec7-a2d4-4518-a3f7-4b84dfb7b9d6"
